File: SwitchingBoard.brd (EAGLE design)
At the start: 160 x 100 mm, 38 parts, among them K1 351, T1 BT148, T2 TICP206, T3 BT136, T4 BT136

Commit message: Updated schematics and parts for the switching board.
Parts:
- added C10, C11, C12: 10nF, rcl:C102-043X133
- added C8, C9: 10nF, rcl:C150-054X183
- added R12, R15: 39, rcl:0207/7
- added R13, R16: 360, rcl:0207/7
- added R14, R17: 390, rcl:0207/7
- added X2, X5: (no value), con-wago-500:W237-102
- C2: device rcl:C225-108X268 -> rcl:C225-062X268
- C7: device rcl:C025-024X044 -> rcl:C150-054X183
- R10: value 360 -> 390
- R11: value 360 -> 39
- moved C7 372.2 mm to (116.8, 81.3), turned to 180 degrees
- moved R10 356.1 mm to (118.1, 90.2), turned to 270 degrees
- moved R9 344.5 mm to (132.1, 77.5), turned to 90 degrees
- moved X9 319.2 mm to (139.7, 86.4), turned to 90 degrees
- moved OK1 300.7 mm to (128.3, 88.9), turned to 90 degrees
- moved R11 297.3 mm to (110.5, 5.08), turned to 90 degrees
- moved R7 270.4 mm to (87.6, 31.8), turned to 90 degrees
- moved X6 248.6 mm to (151.1, 7.62), turned to 90 degrees
- moved X8 226.1 mm to (116.8, 6.35), turned to 90 degrees
- moved T3 172.0 mm to (152.4, 22.9)
- moved X1 163.9 mm to (108.0, 49.5)
- moved T2 162.6 mm to (106.7, 91.4)
- moved T4 154.1 mm to (120.7, 20.3)
- moved X7 7.62 mm to (108.0, 66.0)
- moved T1 2.54 mm to (55.9, 24.1)
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Connections:
- new net N$15: R13.2, X2.1
- new net N$16: C11.1, C8.1, R11.2
- new net N$17: R14.1, T4.3, X2.2
- new net N$20: C10.1, C9.1, R15.2
- new net N$21: R16.2, X5.1
- new net N$22: R17.1, T3.3, X5.2
- net CONTROL_LIVE: now also R12.1; no longer R11.1, R9.1
- net LIVE: now also R11.1, R13.1, R15.1, R16.1
- net N$11: now also C10.2, C9.2, R17.2, T3.1, X6.1, X6.2; no longer T4.1, X8.1, X8.2
- net N$14: now also C12.1, R12.2, R9.1; no longer R11.2
- net N$8: now also C11.2, C8.2, R14.2, T4.1, X8.1, X8.2; no longer T3.1, X6.1, X6.2
- net TIMEDLIVE: now also C12.2
