File: SwitchingBoard.sch (EAGLE design)
At the start: 38 parts, among them K1 351, T1 BT148, T2 TICP206, T3 BT136, T4 BT136

Commit message: Updated schematics and parts for the switching board.
Parts:
- added C10, C11, C12: 10nF, rcl:C-EU102-043X133
- added C8, C9: 10nF, rcl:C-EU150-054X183
- added R12, R15: 39, rcl:R-EU_0207/7
- added R13, R16: 360, rcl:R-EU_0207/7
- added R14, R17: 390, rcl:R-EU_0207/7
- added X2, X5: (no value), con-wago-500:W237-102
- C2: device rcl:C-EU225-108X268 -> rcl:C-EU225-062X268
- C7: device rcl:C-EU025-024X044 -> rcl:C-EU150-054X183
- R10: value 360 -> 390
- R11: value 360 -> 39
Connections:
- new net N$15: R13.2, X2-1.KL
- new net N$16: C11.1, C8.1, R11.2
- new net N$17: R14.1, T4.G, X2-2.KL
- new net N$20: C10.1, C9.1, R15.2
- new net N$21: R16.2, X5-1.KL
- new net N$22: R17.1, T3.G, X5-2.KL
- net CONTROL_LIVE: now also R12.1; no longer R11.1, R9.1
- net LIVE: now also R11.1, R13.1, R15.1, R16.1
- net N$11: now also C10.2, C9.2, R17.2, T3.A1, X6-1.KL, X6-2.KL; no longer T4.A1, X8-1.KL, X8-2.KL
- net N$14: now also C12.1, R12.2, R9.1; no longer R11.2
- net N$8: now also C11.2, C8.2, R14.2, T4.A1, X8-1.KL, X8-2.KL; no longer T3.A1, X6-1.KL, X6-2.KL
- net TIMEDLIVE: now also C12.2
Other:
- moved on the sheet: C7, K1, R11, T2, T3, T4, X1-1, X1-2, X6-1, X6-2, X7-1, X8-1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
