File: InrushTimer.sch (EAGLE design)
At the start: 72 parts, among them IC1 TLC272D, IC2 555, IC3 4076N, Q1 TIP41C, Q2 TRANSISTOR-FET_2N7002, Q3 TRANSISTOR-FET_2N7002, Q4 TRANSISTOR-FET_2N7002, Q5 TRANSISTOR-FET_2N7002, T1 MMBTA05, U1 ROHM_BY_ELEMENT14_BATCH_1_BU4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

Commit message: Rerouted power supply section and made some space around the pot.
Parts:
- D14: value P6KEXXCTS-P6KE -> P6KEXXCDO15-10V; device diode:P6KEXXCTS-P6KE -> diode:P6KEXXCDO15-10V
- R22, R6, R7: device rcl:R-EU_0207/7 -> rcl:R-EU_0207/2V
Connections:
- net N$14: now also R3.1; no longer R3.2
- net ON_A_SYNC: now also R22.1; no longer R22.2
- net THRESH: now also R11.1; no longer R11.2
- net V12: now also D14.1, R11.2, R22.2; no longer D14.2, R11.1, R22.1
- net ZERO: now also D14.2, R3.2; no longer D14.1, R3.1
Other:
- moved on the sheet: D14, R11, R22, R3
Changed lines of the file:
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@@
 <part name="R13" library="rcl" deviceset="R-EU_" device="0207/2V" value="200K"/>
 <part name="R2" library="rcl" deviceset="R-EU_" device="0207/7" value="27K"/>
-<part name="R7" library="rcl" deviceset="R-EU_" device="0207/7" value="51K"/>
-<part name="R6" library="rcl" deviceset="R-EU_" device="0207/7" value="22K"/>
+<part name="R7" library="rcl" deviceset="R-EU_" device="0207/2V" value="51K"/>
+<part name="R6" library="rcl" deviceset="R-EU_" device="0207/2V" value="22K"/>
 <part name="R3" library="rcl" deviceset="R-EU_" device="0207/2V" value="10K"/>
 <part name="C10" library="rcl" deviceset="C-EU" device="C0805K" value="10pF (DNF)"/>
@@
 <part name="D12" library="diode" deviceset="1N4148" device="DO35-7"/>
 <part name="D8" library="diode" deviceset="1N4148" device="DO35-10" value="1N4148DO35-10"/>
-<part name="R22" library="rcl" deviceset="R-EU_" device="0207/7" value="200K"/>
+<part name="R22" library="rcl" deviceset="R-EU_" device="0207/2V" value="200K"/>
 <part name="R23" library="rcl" deviceset="R-EU_" device="0207/7" value="200K"/>
 <part name="D9" library="diode" deviceset="1N4148" device="DO35-7"/>
@@
 <part name="D3" library="diode" deviceset="DIODE-" device="DO34-7" value="5082-2800"/>
 <part name="U$1" library="SHoleLib" deviceset="TLP268J" device=""/>
-<part name="D14" library="diode" deviceset="P6KEXXC" device="TS-P6KE" value="P6KEXXCTS-P6KE"/>
+<part name="D14" library="diode" deviceset="P6KEXXC" device="DO15-10V" value="P6KEXXCDO15-10V"/>
 <part name="Q1" library="transistor-power" deviceset="TIP41C" device=""/>
 </parts>
@@
 <instance part="D5" gate="G$1" x="-66.04" y="93.98" rot="R90"/>
 <instance part="R9" gate="G$1" x="-38.1" y="45.72" rot="R90"/>
-<instance part="R11" gate="G$1" x="0" y="60.96" rot="R270"/>
+<instance part="R11" gate="G$1" x="0" y="60.96" rot="R90"/>
 <instance part="R12" gate="G$1" x="0" y="45.72" rot="R90"/>
 <instance part="IC3" gate="A" x="223.52" y="-7.62"/>
@@
 <instance part="R7" gate="G$1" x="35.56" y="-60.96" rot="R270"/>
 <instance part="R6" gate="G$1" x="7.62" y="-60.96" rot="R90"/>
-<instance part="R3" gate="G$1" x="-73.66" y="-76.2" rot="R90"/>
+<instance part="R3" gate="G$1" x="-73.66" y="-76.2" rot="R270"/>
 <instance part="C10" gate="G$1" x="45.72" y="58.42"/>
 <instance part="D4" gate="G$1" x="-73.66" y="81.28"/>
@@
 <attribute name="NAME" x="261.62" y="17.2974" size="1.778" layer="95" rot="R180"/>
 </instance>
-<instance part="R22" gate="G$1" x="269.24" y="45.72" rot="R270"/>
+<instance part="R22" gate="G$1" x="269.24" y="45.72" rot="R90"/>
 <instance part="R23" gate="G$1" x="276.86" y="45.72" rot="R270"/>
 <instance part="D9" gate="G$1" x="264.16" y="12.7" smashed="yes" rot="R180">
@@
 <instance part="D3" gate="G$1" x="-22.86" y="60.96" rot="R270"/>
 <instance part="U$1" gate="G$1" x="368.3" y="7.62"/>
-<instance part="D14" gate="1" x="-53.34" y="-20.32" rot="R90"/>
+<instance part="D14" gate="1" x="-53.34" y="-17.78" rot="R270"/>
 <instance part="Q1" gate="1" x="-81.28" y="-5.08"/>
 </instances>
@@
 <label x="-68.072" y="-11.684" size="1.778" layer="95"/>
 <pinref part="C3" gate="G$1" pin="+"/>
-<pinref part="D14" gate="1" pin="2"/>
-<wire x1="-53.34" y1="-12.7" x2="-53.34" y2="-15.24" width="0.1524" layer="91"/>
 <pinref part="Q1" gate="1" pin="E"/>
 <wire x1="-78.74" y1="-10.16" x2="-78.74" y2="-12.7" width="0.1524" layer="91"/>
+<pinref part="D14" gate="1" pin="1"/>
+<wire x1="-53.34" y1="-15.24" x2="-53.34" y2="-12.7" width="0.1524" layer="91"/>
 </segment>
 <segment>
@@
 <label x="-10.16" y="68.58" size="1.778" layer="95"/>
 <wire x1="0" y1="68.58" x2="-10.16" y2="68.58" width="0.1524" layer="91"/>
-<pinref part="R11" gate="G$1" pin="1"/>
+<pinref part="R11" gate="G$1" pin="2"/>
 <wire x1="0" y1="66.04" x2="0" y2="68.58" width="0.1524" layer="91"/>
 </segment>
 <segment>
-<pinref part="R22" gate="G$1" pin="1"/>
-<wire x1="269.24" y1="50.8" x2="269.24" y2="55.88" width="0.1524" layer="91"/>
-<wire x1="269.24" y1="55.88" x2="276.86" y2="55.88" width="0.1524" layer="91"/>
-<wire x1="269.24" y1="55.88" x2="261.62" y2="55.88" width="0.1524" layer="91"/>
-<junction x="269.24" y="55.88"/>
+<wire x1="276.86" y1="55.88" x2="269.24" y2="55.88" width="0.1524" layer="91"/>
 <label x="261.62" y="55.88" size="1.778" layer="95"/>
 <pinref part="R23" gate="G$1" pin="1"/>
+<wire x1="269.24" y1="55.88" x2="261.62" y2="55.88" width="0.1524" layer="91"/>
 <wire x1="276.86" y1="50.8" x2="276.86" y2="55.88" width="0.1524" layer="91"/>
+<pinref part="R22" gate="G$1" pin="2"/>
+<wire x1="269.24" y1="50.8" x2="269.24" y2="55.88" width="0.1524" layer="91"/>
+<junction x="269.24" y="55.88"/>
 </segment>
 <segment>
@@
 <wire x1="-119.38" y1="-25.4" x2="-109.22" y2="-25.4" width="0.1524" layer="91"/>
 <junction x="-109.22" y="-25.4"/>
-<pinref part="D14" gate="1" pin="1"/>
-<wire x1="-53.34" y1="-22.86" x2="-53.34" y2="-25.4" width="0.1524" layer="91"/>
+<pinref part="D14" gate="1" pin="2"/>
+<wire x1="-53.34" y1="-25.4" x2="-53.34" y2="-22.86" width="0.1524" layer="91"/>
 </segment>
 <segment>
@@
 <pinref part="D13" gate="G$1" pin="A"/>
 <pinref part="D2" gate="G$1" pin="A"/>
-<pinref part="R3" gate="G$1" pin="1"/>
+<pinref part="R3" gate="G$1" pin="2"/>
 <wire x1="-73.66" y1="-81.28" x2="-73.66" y2="-88.9" width="0.1524" layer="91"/>
 <junction x="-73.66" y="-88.9"/>
@@
 <pinref part="R12" gate="G$1" pin="2"/>
 <wire x1="0" y1="50.8" x2="0" y2="53.34" width="0.1524" layer="91"/>
-<pinref part="R11" gate="G$1" pin="2"/>
+<pinref part="R11" gate="G$1" pin="1"/>
 <wire x1="0" y1="55.88" x2="0" y2="53.34" width="0.1524" layer="91"/>
 <junction x="0" y="53.34"/>
@@
 <pinref part="D11" gate="G$1" pin="A"/>
 <wire x1="266.7" y1="-5.08" x2="269.24" y2="-5.08" width="0.1524" layer="91"/>
-<pinref part="R22" gate="G$1" pin="2"/>
 <wire x1="269.24" y1="-5.08" x2="269.24" y2="17.78" width="0.1524" layer="91"/>
 <wire x1="269.24" y1="17.78" x2="269.24" y2="27.94" width="0.1524" layer="91"/>
 <pinref part="D8" gate="G$1" pin="A"/>
-<wire x1="269.24" y1="27.94" x2="269.24" y2="40.64" width="0.1524" layer="91"/>
 <wire x1="266.7" y1="17.78" x2="269.24" y2="17.78" width="0.1524" layer="91"/>
 <junction x="269.24" y="17.78"/>
@@
 <pinref part="SJ1" gate="1" pin="1"/>
 <wire x1="266.7" y1="27.94" x2="269.24" y2="27.94" width="0.1524" layer="91"/>
-<junction x="269.24" y="27.94"/>
 <wire x1="269.24" y1="-12.7" x2="269.24" y2="-5.08" width="0.1524" layer="91"/>
 <pinref part="C15" gate="G$1" pin="2"/>
+<pinref part="R22" gate="G$1" pin="1"/>
+<wire x1="269.24" y1="40.64" x2="269.24" y2="27.94" width="0.1524" layer="91"/>
+<junction x="269.24" y="27.94"/>
 </segment>
 </net>
@@
 <wire x1="-73.66" y1="-60.96" x2="-73.66" y2="-63.5" width="0.1524" layer="91"/>
 <pinref part="D13" gate="G$1" pin="C"/>
-<pinref part="R3" gate="G$1" pin="2"/>
+<pinref part="R3" gate="G$1" pin="1"/>
 <wire x1="-73.66" y1="-71.12" x2="-73.66" y2="-63.5" width="0.1524" layer="91"/>
 </segment>
